Commit message: Addressed the feedback comments

File: my_robot/urdf/my_robot.xacro (robot description, xacro)
@@ -179,3 +179,11 @@
   <child link="hokuyo"/>
   </joint>
+  <!-- optical camera -->
+  <link name="camera_link_optical">
+  </link>
+  <joint name="camera_optical_joint" type="fixed">
+    <origin xyz="0 0 0" rpy="-1.5707 0 -1.5707"/>
+    <parent link="camera"/>
+    <child link="camera_link_optical"/>
+  </joint>
 </robot>
